File: kicad/branchControllerPCB.sch (KiCad schematic (older format))
At the start: 7 parts, among them J1 RJ45, J2 RJ45, U1 Teensy3.2, U2 SN74HCT245N Level Shifter

Commit message: finished the schematics in kicad
Parts:
- added J3: Adafruit 4400 32x128 OLED, Connector_PinSocket_2.54mm:PinSocket_1x06_P2.54mm_Vertical, symbol branchController:Adafruit_4400_OLED
- added U3: TSOP34438 IR SENSOR, OptoDevice:Vishay_MOLD-3Pin, symbol Interface_Optical:TSOP343xx
- added U4: WIZ850io Ethernet, branchController:WIZ850io, symbol branchController:WIZ850io
- D1: footprint (none) -> LED_THT:LED_D5.0mm
- J1, J2: value RJ45 -> RJ45 AE10388-ND; footprint (none) -> branchController:ASSMANN_A-2004-1-4-LP-N-R
- R1: footprint (none) -> Resistor_THT:R_Axial_DIN0411_L9.9mm_D3.6mm_P7.62mm_Vertical
- RN1: footprint (none) -> branchController:4116R-1-101LF
- U2: footprint (none) -> branchController:SN74HCT245N
Connections:
- net +3V3: now also U3.3 (Vs), U4.8 (3.3V_1), U4.9 (3.3V_2); no longer U2.20 (VCC)
- net GND: now also J3.GND (4), U3.2 (GND), U4.1 (GND_1), U4.2 (GND_2), U4.7 (GND_3)
- net SCN: now reaches U1.12 (10_TX2_CS_PWM)
- net SCN: now also U4.5 (SCNN)
- net MOSI: now reaches U1.13 (11_DOUT)
- net MOSI: now also U4.3 (MOSI)
- net MISO: now reaches U1.14 (12_DIN)
- net MISO: now also U4.12 (MISO)
- net SCLK: now reaches U1.20 (13_LED_SCK)
- net SCLK: now also U4.4 (SCLK)
- net I2CSDA: now reaches U1.25 (18_A4_SDA0_Touch)
- net I2CSDA: now also J3.SDA (1)
- net I2CSCL: now reaches U1.26 (19_A5_SCL0_Touch)
- net I2CSCL: now also J3.SCL (2)
- net IR: now reaches U1.3 (1_TX1_Touch)
- net IR: now also U3.1 (OUT)
- net +5V: now reaches U1.33 (Vin)
- net +5V: now also U2.20 (VCC), J3.VIN (6)
- no-connect marks 0 -> 38

Commit message: finished designing prototype circuit board
Parts:
- J3: footprint Connector_PinSocket_2.54mm:PinSocket_1x06_P2.54mm_Vertical -> branchController:AdaFruit4400LED
Connections:
- net IR: now also U1.5 (3_TX_PWM); no longer U1.3 (1_TX1_Touch)
Changed lines of the file:
@@
 	1    0    0    -1
 $EndComp
-Text Label 7050 1550 0    50   ~ 0
+Text Label 7050 1750 0    50   ~ 0
 IR
-Wire Wire Line
-	7050 1550 7450 1550
 Text Label 9600 5750 2    50   ~ 0
 IR
@@
 	9600 5750 9250 5750
 $Comp
-L power:GND #PWR?
+L power:GND #PWR0104
 U 1 1 5E054B02
 P 9550 5950
-F 0 "#PWR?" H 9550 5700 50  0001 C CNN
+F 0 "#PWR0104" H 9550 5700 50  0001 C CNN
 F 1 "GND" H 9555 5777 50  0000 C CNN
 F 2 "" H 9550 5950 50  0001 C CNN
@@
 	9550 5950 9250 5950
 $Comp
-L power:+3.3V #PWR?
+L power:+3.3V #PWR0109
 U 1 1 5E059FFC
 P 9550 5550
-F 0 "#PWR?" H 9550 5400 50  0001 C CNN
+F 0 "#PWR0109" H 9550 5400 50  0001 C CNN
 F 1 "+3.3V" H 9565 5723 50  0000 C CNN
 F 2 "" H 9550 5550 50  0001 C CNN
@@
 	3900 4850 3450 4850
 $Comp
-L power:GND #PWR?
+L power:GND #PWR0110
 U 1 1 5E084244
 P 3750 5350
-F 0 "#PWR?" H 3750 5100 50  0001 C CNN
+F 0 "#PWR0110" H 3750 5100 50  0001 C CNN
 F 1 "GND" H 3755 5177 50  0000 C CNN
 F 2 "" H 3750 5350 50  0001 C CNN
@@
 	3750 4750 3750 5350
 $Comp
-L power:GND #PWR?
+L power:GND #PWR0111
 U 1 1 5E08D650
 P 5350 5400
-F 0 "#PWR?" H 5350 5150 50  0001 C CNN
+F 0 "#PWR0111" H 5350 5150 50  0001 C CNN
 F 1 "GND" H 5355 5227 50  0000 C CNN
 F 2 "" H 5350 5400 50  0001 C CNN
@@
 	5350 4650 5200 4650
 $Comp
-L power:+3.3V #PWR?
+L power:+3.3V #PWR0112
 U 1 1 5E0914AE
 P 5600 4500
-F 0 "#PWR?" H 5600 4350 50  0001 C CNN
+F 0 "#PWR0112" H 5600 4350 50  0001 C CNN
 F 1 "+3.3V" H 5615 4673 50  0000 C CNN
 F 2 "" H 5600 4500 50  0001 C CNN
@@
 NoConn ~ 3900 5150
 $Comp
-L power:+5V #PWR?
+L power:+5V #PWR0113
 U 1 1 5E0A7C46
 P 2750 1200
-F 0 "#PWR?" H 2750 1050 50  0001 C CNN
+F 0 "#PWR0113" H 2750 1050 50  0001 C CNN
 F 1 "+5V" H 2765 1373 50  0000 C CNN
 F 2 "" H 2750 1200 50  0001 C CNN
@@
 	1800 1200 2750 1200
 $Comp
-L power:+5V #PWR?
+L power:+5V #PWR0114
 U 1 1 5E0C0175
 P 9800 3650
-F 0 "#PWR?" H 9800 3500 50  0001 C CNN
+F 0 "#PWR0114" H 9800 3500 50  0001 C CNN
 F 1 "+5V" H 9815 3823 50  0000 C CNN
 F 2 "" H 9800 3650 50  0001 C CNN
@@
 F 0 "J3" H 1668 4225 50  0000 C CNN
 F 1 "Adafruit 4400 32x128 OLED" H 1668 4316 50  0000 C CNN
-F 2 "Connector_PinSocket_2.54mm:PinSocket_1x06_P2.54mm_Vertical" H 1750 4750 50  0001 C CNN
+F 2 "branchController:AdaFruit4400LED" H 1750 4750 50  0001 C CNN
 F 3 "https://www.adafruit.com/product/4440" H 1750 4750 50  0001 C CNN
 	1    1750 4750
@@
 $EndComp
 $Comp
-L power:+5V #PWR?
+L power:+5V #PWR0115
 U 1 1 5E0E4E6C
 P 2450 4450
-F 0 "#PWR?" H 2450 4300 50  0001 C CNN
+F 0 "#PWR0115" H 2450 4300 50  0001 C CNN
 F 1 "+5V" H 2465 4623 50  0000 C CNN
 F 2 "" H 2450 4450 50  0001 C CNN
@@
 $EndComp
 $Comp
-L power:GND #PWR?
+L power:GND #PWR0116
 U 1 1 5E0E5253
 P 2450 4650
-F 0 "#PWR?" H 2450 4400 50  0001 C CNN
+F 0 "#PWR0116" H 2450 4400 50  0001 C CNN
 F 1 "GND" H 2455 4477 50  0000 C CNN
 F 2 "" H 2450 4650 50  0001 C CNN
@@
 	7050 3850 7450 3850
 NoConn ~ 7450 1450
-NoConn ~ 7450 1750
 NoConn ~ 7450 1850
 NoConn ~ 7450 2350
@@
 NoConn ~ 9450 1450
 NoConn ~ 9450 1350
+NoConn ~ 7450 1550
+Wire Wire Line
+	7450 1750 7050 1750
 $EndSCHEMATC
