File: kicad/branchControllerPCB.kicad_pcb (KiCad board)
At the start: 4 copper layers, 102.9 x 72.4 mm, 10 parts, among them J1 RJ45 AE10388-ND, J2 RJ45 AE10388-ND, J3 Adafruit 4400 32x128 OLED, U2 Level Shifter, U4 WIZ850io Ethernet

Commit message: tweaks and improvements to PCB
Parts:
- moved IR 52.6 mm to (200.7, 87.6)
Routing:
- net /IR: track 96.0 -> 43.8 mm
- net +3V3: track 30.3 -> 0.00 mm
- net /I2CSDA: track 30.2 -> 33.2 mm
- net /SCN: track 36.3 -> 37.0 mm
- net /SCLK: track 27.3 -> 27.8 mm
Other:
- board size 102.9 x 72.4 mm -> 107.9 x 74.9 mm
- board text added: "1 2 3 4"
- board text added: "5 6 7 8"
- board text added: "BRANCH CONTROLLER PROTOTYPE 0.1 JOEL SPOLSKY blinkylights.blog"
- board text removed: "BRANCH CONTROLLER PROTOTYPE 0.1 JOEL SPOLSKY"

Commit message: final kicad
Routing:
- net /SCLK: track 27.8 -> 26.6 mm
Changed lines of the file:
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@@
     (thickness 1.6)
     (drawings 15)
-    (tracks 172)
+    (tracks 168)
     (zones 0)
     (modules 10)
@@
       (outputformat 1)
       (mirror false)
-      (drillshape 1)
+      (drillshape 0)
       (scaleselection 1)
-      (outputdirectory ""))
+      (outputdirectory "gerber/"))
   )
   (net 0 "")
@@
   (module teensy:Teensy30_31_32_LC (layer F.Cu)
     (at 187.96 120.65 90)
-    (fp_text reference "TEENSY 3.2" (at -6.35 0 90) (layer F.SilkS)
+    (fp_text reference "TEENSY 3.2" (at -1.27 0 180) (layer F.SilkS)
       (effects (font (size 1 1) (thickness 0.15)))
     )
@@
   (segment (start 222.25 109.22) (end 229.362 109.22) (width 0.25) (layer F.Cu) (net 18))
   (segment (start 222.25 111.76) (end 229.362 111.76) (width 0.25) (layer F.Cu) (net 19))
-  (segment (start 181.139999 104.939999) (end 180.34 104.14) (width 0.25) (layer In1.Cu) (net 23))
-  (segment (start 181.465001 105.265001) (end 181.139999 104.939999) (width 0.25) (layer In1.Cu) (net 23))
-  (segment (start 181.465001 109.760001) (end 181.465001 105.265001) (width 0.25) (layer In1.Cu) (net 23))
-  (segment (start 180.089997 110.345001) (end 180.880001 110.345001) (width 0.25) (layer In1.Cu) (net 23))
+  (segment (start 177.8 111.219999) (end 177.8 106.68) (width 0.25) (layer In1.Cu) (net 23))
+  (segment (start 178.640993 114.249497) (end 177.8 111.219999) (width 0.25) (layer In1.Cu) (net 23))
+  (segment (start 176.53 118.11) (end 178.640993 114.249497) (width 0.25) (layer In1.Cu) (net 23))
+  (segment (start 177.8 106.68) (end 180.34 104.14) (width 0.25) (layer In1.Cu) (net 23))
+  (segment (start 171.006898 120.65) (end 171.893102 120.65) (width 0.25) (layer In1.Cu) (net 23))
+  (segment (start 171.893102 120.65) (end 175.26 118.11) (width 0.25) (layer In1.Cu) (net 23))
+  (segment (start 175.26 118.11) (end 176.53 118.11) (width 0.25) (layer In1.Cu) (net 23))
   (segment (start 170.292499 121.364399) (end 171.006898 120.65) (width 0.25) (layer In1.Cu) (net 23))
-  (segment (start 179.214999 111.219999) (end 180.089997 110.345001) (width 0.25) (layer In1.Cu) (net 23))
-  (segment (start 176.53 118.11) (end 179.07 115.57) (width 0.25) (layer In1.Cu) (net 23))
-  (segment (start 175.26 118.11) (end 176.53 118.11) (width 0.25) (layer In1.Cu) (net 23))
-  (segment (start 171.893102 120.65) (end 175.26 118.11) (width 0.25) (layer In1.Cu) (net 23))
-  (segment (start 171.006898 120.65) (end 171.893102 120.65) (width 0.25) (layer In1.Cu) (net 23))
   (segment (start 170.292499 123.302499) (end 170.292499 121.364399) (width 0.25) (layer In1.Cu) (net 23))
-  (segment (start 179.07 115.57) (end 179.214999 111.219999) (width 0.25) (layer In1.Cu) (net 23))
-  (segment (start 180.880001 110.345001) (end 181.465001 109.760001) (width 0.25) (layer In1.Cu) (net 23))
   (segment (start 171.45 124.46) (end 170.292499 123.302499) (width 0.25) (layer In1.Cu) (net 23))
   (segment (start 194.780001 104.939999) (end 195.58 104.14) (width 0.25) (layer In1.Cu) (net 26))

Commit message: Tweaked PCB dimensions
No electrical changes
Parts:
- 100 OHM: renamed from RN1
- renumbered U2 to SN74HCT245N
Other:
- board size 107.9 x 74.9 mm -> 107.9 x 69.9 mm
- board text added: "BRANCH CONTROLLER PROTOTYPE 0.2 JOEL SPOLSKY blinkylights.blog"
- board text added: "USB"
- board text added: "github.com/jspolsky/branchController2"
- board text added: "https://github.com/jspolsky/branchController2"
- board text removed: "BRANCH CONTROLLER PROTOTYPE 0.1 JOEL SPOLSKY blinkylights.blog"
Changed lines of the file:
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@@
   (general
     (thickness 1.6)
-    (drawings 15)
+    (drawings 22)
     (tracks 168)
     (zones 0)
@@
   (layers
     (0 F.Cu power hide)
-    (1 In1.Cu signal)
+    (1 In1.Cu signal hide)
     (2 In2.Cu signal hide)
     (31 B.Cu power hide)
@@
     (34 B.Paste user hide)
     (35 F.Paste user hide)
-    (36 B.SilkS user hide)
+    (36 B.SilkS user)
     (37 F.SilkS user)
     (38 B.Mask user hide)
@@
     (43 Eco2.User user hide)
     (44 Edge.Cuts user)
-    (45 Margin user)
+    (45 Margin user hide)
     (46 B.CrtYd user hide)
     (47 F.CrtYd user hide)
@@
       (drillshape 0)
       (scaleselection 1)
-      (outputdirectory "gerber/"))
+      (outputdirectory "/Users/spolsky/Dropbox/Arduino/branchController2/gerber/"))
   )
   (net 0 "")
@@
   (module branchController:SN74HCT245N (layer F.Cu)
     (at 222.25 111.76)
-    (fp_text reference U2 (at -5.08 -3.81 90) (layer F.SilkS)
+    (fp_text reference SN74HCT245N (at -5.08 -7.62 90) (layer F.SilkS)
       (effects (font (size 1 1) (thickness 0.15)))
     )
@@
   (module branchController:4116R-1-101LF (layer F.Cu)
     (at 237.49 111.76)
-    (fp_text reference RN1 (at -6.35 -3.81 270) (layer F.SilkS)
-      (effects (font (size 1 1) (thickness 0.15)))
-    )
-    (fp_text value "RES ARRAY" (at -3.81 -6.35 90) (layer F.SilkS)
+    (fp_text reference "100 OHM" (at -5.08 -6.35 270) (layer F.SilkS)
+      (effects (font (size 1 1) (thickness 0.15)))
+    )
+    (fp_text value "RES ARRAY" (at -2.54 -6.35 90) (layer F.SilkS)
       (effects (font (size 1 1) (thickness 0.15)))
     )
@@
   (module branchController:ASSMANN_A-2004-1-4-LP-N-R (layer F.Cu)
     (at 229.87 130.81)
-    (fp_text reference J2 (at -5.78656 -11.5496) (layer F.SilkS)
+    (fp_text reference J2 (at -1.27 -3.81) (layer F.SilkS)
       (effects (font (size 1 1) (thickness 0.015)))
     )
@@
   (module branchController:ASSMANN_A-2004-1-4-LP-N-R (layer F.Cu)
     (at 209.55 130.81)
-    (fp_text reference J1 (at -5.78656 -11.5496) (layer F.SilkS)
+    (fp_text reference J1 (at -1.27 -3.81) (layer F.SilkS)
       (effects (font (size 1 1) (thickness 0.015)))
     )
@@
     )
   )
-  (gr_text "5  6  7  8" (at 229.87 142.24) (layer F.SilkS)
+  (gr_text github.com/jspolsky/branchController2 (at 245.11 106.68 90) (layer F.SilkS)
     (effects (font (size 1 1) (thickness 0.15)))
   )
-  (gr_text "1  2  3  4\n" (at 209.55 142.24) (layer F.SilkS)
+  (gr_text USB (at 187.96 137.16) (layer B.SilkS)
+    (effects (font (size 1 1) (thickness 0.15)) (justify mirror))
+  )
+  (gr_text ETHERNET (at 161.29 137.16) (layer B.SilkS)
+    (effects (font (size 1 1) (thickness 0.15)) (justify mirror))
+  )
+  (gr_text https://github.com/jspolsky/branchController2 (at 195.58 76.2) (layer B.SilkS)
+    (effects (font (size 1 1) (thickness 0.15)) (justify mirror))
+  )
+  (gr_arc (start 142.24 138.43) (end 140.97 138.43) (angle -90) (layer Edge.Cuts) (width 0.05))
+  (gr_arc (start 247.65 138.43) (end 247.65 139.7) (angle -90) (layer Edge.Cuts) (width 0.05))
+  (gr_arc (start 140.97 69.85) (end 140.97 74.93) (angle -90) (layer Edge.Cuts) (width 0.05))
+  (gr_arc (start 248.92 69.85) (end 243.84 69.85) (angle -90) (layer Edge.Cuts) (width 0.05))
+  (gr_text "5  6  7  8" (at 229.87 118.11) (layer F.SilkS)
     (effects (font (size 1 1) (thickness 0.15)))
   )
-  (gr_text ETHERNET (at 161.29 142.24) (layer F.SilkS)
+  (gr_text "1  2  3  4\n" (at 209.55 118.11) (layer F.SilkS)
     (effects (font (size 1 1) (thickness 0.15)))
   )
-  (gr_text ETHERNET (at 163.83 142.24) (layer B.Cu)
-    (effects (font (size 1.5 1.5) (thickness 0.3)) (justify mirror))
-  )
-  (gr_line (start 140.97 144.78) (end 140.97 69.85) (layer Edge.Cuts) (width 0.05))
-  (gr_line (start 248.92 144.78) (end 140.97 144.78) (layer Edge.Cuts) (width 0.05))
-  (gr_line (start 248.92 69.85) (end 248.92 144.78) (layer Edge.Cuts) (width 0.05))
-  (gr_line (start 140.97 69.85) (end 248.92 69.85) (layer Edge.Cuts) (width 0.05))
-  (gr_circle (center 147.32 76.2) (end 150.7236 76.2) (layer Edge.Cuts) (width 0.05))
-  (gr_circle (center 243.332 76.2) (end 246.7356 76.2) (layer Edge.Cuts) (width 0.05))
-  (gr_text "BRANCH CONTROLLER PROTOTYPE 0.1\nJOEL SPOLSKY\nblinkylights.blog" (at 218.44 78.74) (layer F.SilkS)
+  (gr_text ETHERNET (at 146.05 124.46 90) (layer F.SilkS)
     (effects (font (size 1 1) (thickness 0.15)))
+  )
+  (gr_line (start 140.97 138.43) (end 140.97 74.93) (layer Edge.Cuts) (width 0.05))
+  (gr_line (start 247.65 139.7) (end 142.24 139.7) (layer Edge.Cuts) (width 0.05))
+  (gr_line (start 248.92 74.93) (end 248.92 138.43) (layer Edge.Cuts) (width 0.05))
+  (gr_line (start 146.05 69.85) (end 243.84 69.85) (layer Edge.Cuts) (width 0.05))
+  (gr_circle (center 147.32 76.2) (end 149.479 76.2) (layer Edge.Cuts) (width 0.05))
+  (gr_circle (center 243.332 76.2) (end 245.491 76.2) (layer Edge.Cuts) (width 0.05))
+  (gr_text "BRANCH CONTROLLER PROTOTYPE 0.2\nJOEL SPOLSKY\nblinkylights.blog" (at 215.9 78.74) (layer F.SilkS)
+    (effects (font (size 1.6 1.6) (thickness 0.3)))
   )
   (gr_text OLED (at 172.72 87.63) (layer F.SilkS)
@@
     (polygon
       (pts
-        (xy 246.38 144.78) (xy 143.51 144.78) (xy 143.51 72.39) (xy 246.38 72.39)
+        (xy 248.92 139.7) (xy 140.97 139.7) (xy 140.97 69.85) (xy 248.92 69.85)
       )
     )
@@
     (polygon
       (pts
-        (xy 246.38 144.78) (xy 143.51 144.78) (xy 143.51 72.39) (xy 246.38 72.39)
+        (xy 248.92 139.7) (xy 140.97 139.7) (xy 140.97 69.85) (xy 248.92 69.85)
       )
     )
-  )
-  (zone (net 2) (net_name GND) (layer F.Cu) (hatch edge 0.508)
-    (connect_pads (clearance 0.508))
-    (min_thickness 0.254)
-    (fill yes (arc_segments 32) (thermal_gap 0.508) (thermal_bridge_width 0.508))
-    (polygon
-      (pts
-        (xy 248.92 144.78) (xy 140.97 144.78) (xy 140.97 69.85) (xy 248.92 69.85)
-      )
-    )
-  )
-  (zone (net 36) (net_name +3V3) (layer B.Cu) (hatch edge 0.508)
-    (connect_pads (clearance 0.508))
-    (min_thickness 0.254)
-    (fill yes (arc_segments 32) (thermal_gap 0.508) (thermal_bridge_width 0.508))
-    (polygon
-      (pts
-        (xy 248.92 144.78) (xy 140.97 144.78) (xy 140.97 69.85) (xy 248.92 69.85)
-      )
-    )
